File: Hardware/Adept_BLE.kicad_sch (KiCad schematic)
At the start: 0 parts

Commit message: update the schematics
Parts:
- added J4: Conn_01x02_Pin, symbol Adept_BLE_symbols:Conn_01x02_Pin
- added J5, J6: Conn_01x01_Pad, symbol Adept_BLE_symbols:Conn_01x01_Pad
- added SW8: PCM12SMTR, Adept_BLE_footprints:PCM12SMTR, symbol Adept_BLE_symbols:PCM12SMTR
Other:
- added sheet PMW3610 (pmw3610.kicad_sch)
- added sheet nRF52840 (nrf52840.kicad_sch)

Commit message: update the schematics
Parts:
- removed J4: Conn_01x02_Pin, symbol Adept_BLE_symbols:Conn_01x02_Pin
- removed J5, J6: Conn_01x01_Pad, symbol Adept_BLE_symbols:Conn_01x01_Pad
- removed SW8: PCM12SMTR, Adept_BLE_footprints:PCM12SMTR, symbol Adept_BLE_symbols:PCM12SMTR
