File: Hardware/pmw3610.kicad_sch (KiCad schematic)
At the start: 11 parts, among them U2 PMW3610DM-SUDU, U3 TLV74318P

Commit message: update the schematics
Parts:
- C7: renamed from C2; value 1u -> 1u/X7R
- renumbered C7 to C1, C8 to C2, C4 to C3, C5 to C4, C3 to C5, C1 to C6, C6 to C8, U3 to U1
Changed lines of the file:
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@@
 		(on_board yes)
 		(dnp no)
-		(property "Reference" "C7"
+		(property "Reference" "C1"
 			(at 193.802 76.2 0)
 			(effects
@@
 			(project ""
 				(path "/17196d55-372c-4b54-86c6-5349d815bf70/c0fc51d6-1fb2-4ff4-a0b4-5fea483719d0"
-					(reference "C7")
+					(reference "C1")
 					(unit 1)
 				)
@@
 		(on_board yes)
 		(dnp no)
-		(property "Reference" "C6"
+		(property "Reference" "C8"
 			(at 182.372 115.57 0)
 			(effects
@@
 			(project ""
 				(path "/17196d55-372c-4b54-86c6-5349d815bf70/c0fc51d6-1fb2-4ff4-a0b4-5fea483719d0"
-					(reference "C6")
+					(reference "C8")
 					(unit 1)
 				)
@@
 		(on_board yes)
 		(dnp no)
-		(fields_autoplaced yes)
-		(property "Reference" "#PWR019"
+		(property "Reference" "#PWR02"
 			(at 214.63 72.39 0)
 			(effects
@@
 		)
 		(property "Value" "+1V8"
-			(at 214.63 63.5 0)
+			(at 214.63 64.262 0)
 			(effects
 				(font
@@
 			(project "Adept_BLE"
 				(path "/17196d55-372c-4b54-86c6-5349d815bf70/c0fc51d6-1fb2-4ff4-a0b4-5fea483719d0"
-					(reference "#PWR019")
+					(reference "#PWR02")
 					(unit 1)
 				)
@@
 		(on_board yes)
 		(dnp no)
-		(property "Reference" "C1"
+		(property "Reference" "C6"
 			(at 78.232 106.68 0)
 			(effects
@@
 			(project ""
 				(path "/17196d55-372c-4b54-86c6-5349d815bf70/c0fc51d6-1fb2-4ff4-a0b4-5fea483719d0"
-					(reference "C1")
+					(reference "C6")
 					(unit 1)
 				)
@@
 		(dnp no)
 		(fields_autoplaced yes)
-		(property "Reference" "U3"
+		(property "Reference" "U1"
 			(at 99.06 93.98 0)
 			(effects
@@
 			(project ""
 				(path "/17196d55-372c-4b54-86c6-5349d815bf70/c0fc51d6-1fb2-4ff4-a0b4-5fea483719d0"
-					(reference "U3")
+					(reference "U1")
 					(unit 1)
 				)
@@
 		(on_board yes)
 		(dnp no)
-		(property "Reference" "C4"
+		(property "Reference" "C3"
 			(at 160.528 90.17 0)
 			(effects
@@
 			(project ""
 				(path "/17196d55-372c-4b54-86c6-5349d815bf70/c0fc51d6-1fb2-4ff4-a0b4-5fea483719d0"
-					(reference "C4")
+					(reference "C3")
 					(unit 1)
 				)
@@
 		(on_board yes)
 		(dnp no)
-		(property "Reference" "#PWR022"
+		(property "Reference" "#PWR09"
 			(at 99.06 123.19 0)
 			(effects
@@
 			(project "Adept_BLE"
 				(path "/17196d55-372c-4b54-86c6-5349d815bf70/c0fc51d6-1fb2-4ff4-a0b4-5fea483719d0"
-					(reference "#PWR022")
+					(reference "#PWR09")
 					(unit 1)
 				)
@@
 		(on_board yes)
 		(dnp no)
-		(fields_autoplaced yes)
-		(property "Reference" "#PWR021"
+		(property "Reference" "#PWR06"
 			(at 81.28 99.06 0)
 			(effects
@@
 		)
 		(property "Value" "+3V3"
-			(at 81.28 90.17 0)
+			(at 81.28 90.932 0)
 			(effects
 				(font
@@
 			(project ""
 				(path "/17196d55-372c-4b54-86c6-5349d815bf70/c0fc51d6-1fb2-4ff4-a0b4-5fea483719d0"
-					(reference "#PWR021")
+					(reference "#PWR06")
 					(unit 1)
 				)
@@
 		(on_board yes)
 		(dnp no)
-		(fields_autoplaced yes)
-		(property "Reference" "#PWR020"
+		(property "Reference" "#PWR07"
 			(at 114.3 99.06 0)
 			(effects
@@
 		)
 		(property "Value" "+1V8"
-			(at 114.3 90.17 0)
+			(at 114.3 90.932 0)
 			(effects
 				(font
@@
 			(project ""
 				(path "/17196d55-372c-4b54-86c6-5349d815bf70/c0fc51d6-1fb2-4ff4-a0b4-5fea483719d0"
-					(reference "#PWR020")
+					(reference "#PWR07")
 					(unit 1)
 				)
@@
 		(on_board yes)
 		(dnp no)
-		(property "Reference" "C8"
+		(property "Reference" "C2"
 			(at 217.678 76.2 0)
 			(effects
@@
 			(project ""
 				(path "/17196d55-372c-4b54-86c6-5349d815bf70/c0fc51d6-1fb2-4ff4-a0b4-5fea483719d0"
-					(reference "C8")
+					(reference "C2")
 					(unit 1)
 				)
@@
 		(on_board yes)
 		(dnp no)
-		(property "Reference" "#PWR017"
+		(property "Reference" "#PWR03"
 			(at 196.85 90.17 0)
 			(effects
@@
 			(project "Adept_BLE"
 				(path "/17196d55-372c-4b54-86c6-5349d815bf70/c0fc51d6-1fb2-4ff4-a0b4-5fea483719d0"
-					(reference "#PWR017")
+					(reference "#PWR03")
 					(unit 1)
 				)
@@
 		(on_board yes)
 		(dnp no)
-		(property "Reference" "#PWR015"
+		(property "Reference" "#PWR011"
 			(at 205.74 132.08 0)
 			(effects
@@
 			(project "Adept_BLE"
 				(path "/17196d55-372c-4b54-86c6-5349d815bf70/c0fc51d6-1fb2-4ff4-a0b4-5fea483719d0"
-					(reference "#PWR015")
+					(reference "#PWR011")
 					(unit 1)
 				)
@@
 		(on_board yes)
 		(dnp no)
-		(property "Reference" "#PWR016"
+		(property "Reference" "#PWR04"
 			(at 214.63 90.17 0)
 			(effects
@@
 			(project "Adept_BLE"
 				(path "/17196d55-372c-4b54-86c6-5349d815bf70/c0fc51d6-1fb2-4ff4-a0b4-5fea483719d0"
-					(reference "#PWR016")
+					(reference "#PWR04")
 					(unit 1)
 				)
@@
 		(on_board yes)
 		(dnp no)
-		(property "Reference" "C3"
+		(property "Reference" "C5"
 			(at 174.752 104.14 0)
 			(effects
@@
 			(project ""
 				(path "/17196d55-372c-4b54-86c6-5349d815bf70/c0fc51d6-1fb2-4ff4-a0b4-5fea483719d0"
-					(reference "C3")
+					(reference "C5")
 					(unit 1)
 				)
@@
 		(on_board yes)
 		(dnp no)
-		(property "Reference" "C5"
+		(property "Reference" "C4"
 			(at 175.514 90.17 0)
 			(effects
@@
 			(project ""
 				(path "/17196d55-372c-4b54-86c6-5349d815bf70/c0fc51d6-1fb2-4ff4-a0b4-5fea483719d0"
-					(reference "C5")
+					(reference "C4")
 					(unit 1)
 				)
@@
 		(on_board yes)
 		(dnp no)
-		(fields_autoplaced yes)
-		(property "Reference" "#PWR023"
+		(property "Reference" "#PWR05"
 			(at 228.6 90.17 0)
 			(effects
@@
 		)
 		(property "Value" "+3V3"
-			(at 228.6 81.28 0)
+			(at 228.6 82.042 0)
 			(effects
 				(font
@@
 			(project "Adept_BLE"
 				(path "/17196d55-372c-4b54-86c6-5349d815bf70/c0fc51d6-1fb2-4ff4-a0b4-5fea483719d0"
-					(reference "#PWR023")
+					(reference "#PWR05")
 					(unit 1)
 				)
@@
 		(on_board yes)
 		(dnp no)
-		(property "Reference" "#PWR013"
+		(property "Reference" "#PWR010"
 			(at 185.42 129.54 0)
 			(effects
@@
 			(project "Adept_BLE"
 				(path "/17196d55-372c-4b54-86c6-5349d815bf70/c0fc51d6-1fb2-4ff4-a0b4-5fea483719d0"
-					(reference "#PWR013")
+					(reference "#PWR010")
 					(unit 1)
 				)
@@
 		(on_board yes)
 		(dnp no)
-		(property "Reference" "C2"
+		(property "Reference" "C7"
 			(at 117.348 106.68 0)
 			(effects
@@
 			)
 		)
-		(property "Value" "1u"
+		(property "Value" "1u/X7R"
 			(at 117.348 109.22 0)
 			(effects
@@
 			(project ""
 				(path "/17196d55-372c-4b54-86c6-5349d815bf70/c0fc51d6-1fb2-4ff4-a0b4-5fea483719d0"
-					(reference "C2")
+					(reference "C7")
 					(unit 1)
 				)
@@
 		(on_board yes)
 		(dnp no)
-		(fields_autoplaced yes)
-		(property "Reference" "#PWR018"
+		(property "Reference" "#PWR01"
 			(at 196.85 72.39 0)
 			(effects
@@
 		)
 		(property "Value" "+3V3"
-			(at 196.85 63.5 0)
+			(at 196.85 64.262 0)
 			(effects
 				(font
@@
 			(project "Adept_BLE"
 				(path "/17196d55-372c-4b54-86c6-5349d815bf70/c0fc51d6-1fb2-4ff4-a0b4-5fea483719d0"
-					(reference "#PWR018")
+					(reference "#PWR01")
 					(unit 1)
 				)
@@
 		(on_board yes)
 		(dnp no)
-		(property "Reference" "#PWR014"
+		(property "Reference" "#PWR08"
 			(at 157.48 106.68 0)
 			(effects
@@
 			(project "Adept_BLE"
 				(path "/17196d55-372c-4b54-86c6-5349d815bf70/c0fc51d6-1fb2-4ff4-a0b4-5fea483719d0"
-					(reference "#PWR014")
-					(unit 1)
-				)
+					(reference "#PWR08")
+					(unit 1)
+				)
