File: Hardware/Adept_BLE.kicad_pcb (KiCad board)
At the start: 2 copper layers, 62 x 65.2 mm, 13 parts, among them J1 Conn_01x07_Pad, J2 Conn_01x07_Pad, SW1 D2LS-21, SW2 D2LS-21, SW3 D2LS-21, SW4 D2LS-21, SW5 D2LS-21, SW6 D2LS-21, SW7 EVQPUC02K, SW8 PCM12SMTR, U1 XIAO-nRF52840-SMD, U2 PMW3610DM-SUDU, U3 TLV74318P

Commit message: update the pcb
Parts:
- added C1: 1u, Adept_BLE_footprints:C_0805, F.Cu at (100.4, 77.8)
- added C2: 1u, Adept_BLE_footprints:C_0805, F.Cu at (100.4, 80.8)
- added C3: 100n/X7R, Adept_BLE_footprints:C_0805, F.Cu at (100.4, 83.8)
- added C4: 10u/X7R, Adept_BLE_footprints:C_0805, F.Cu at (100.4, 86.8)
- added C5: 10n/X7R, Adept_BLE_footprints:C_0805, F.Cu at (100.4, 89.8)
- added C6: 10n, Adept_BLE_footprints:C_0805, F.Cu at (100.4, 92.8)
- added C7: 100n, Adept_BLE_footprints:C_0805, F.Cu at (100.4, 95.8)
- added C8: 100n, Adept_BLE_footprints:C_0805, F.Cu at (100.4, 98.8)
- added J3: Conn_01x01_Pad, Adept_BLE_footprints:Pad_3x2mm, F.Cu at (119.0, 84.6)
- added J4: Conn_01x02_Pin, Adept_BLE_footprints:S2B-PH-K, F.Cu at (112.0, 85.5)
- added J5: Conn_01x01_Pad, Adept_BLE_footprints:Pad_3x2mm, F.Cu at (119.0, 87.6)
- added J6: Conn_01x01_Pad, Adept_BLE_footprints:Pad_3x2mm, F.Cu at (119.0, 90.6)
- added R1: 10k, Adept_BLE_footprints:R_0805, F.Cu at (104.8, 77.7)
- moved SW8 60.3 mm to (110.8, 64.3)
- moved U3 30.1 mm to (108.1, 97.0)
- moved SW7 27.8 mm to (115.6, 73.5)
Connections:
- J1 pad 2: unconnected-(J1-Pin_2-Pad2) -> SW_LB
- J1 pad 3: unconnected-(J1-Pin_3-Pad3) -> SW_LT
- J1 pad 4: unconnected-(J1-Pin_4-Pad4) -> SW_ML
- J1 pad 5: unconnected-(J1-Pin_5-Pad5) -> SW_MR
- J1 pad 6: unconnected-(J1-Pin_6-Pad6) -> SW_RT
- J1 pad 7: unconnected-(J1-Pin_7-Pad7) -> SW_RB
- J2 pad 2: unconnected-(J2-Pin_2-Pad2) -> GND
- J2 pad 3: unconnected-(J2-Pin_3-Pad3) -> +3.3V
- J2 pad 4: unconnected-(J2-Pin_4-Pad4) -> PMW_MOTION
- J2 pad 5: unconnected-(J2-Pin_5-Pad5) -> PMW_SDIO
- J2 pad 6: unconnected-(J2-Pin_6-Pad6) -> PMW_SCLK
- J2 pad 7: unconnected-(J2-Pin_7-Pad7) -> PMW_NCS
- SW1 pad 1: unconnected-(SW1-A-Pad1) -> SW_LB
- SW1 pad 2: unconnected-(SW1-B-Pad2) -> GND
- SW2 pad 1: unconnected-(SW2-A-Pad1) -> SW_LT
- SW2 pad 2: unconnected-(SW2-B-Pad2) -> GND
- SW3 pad 1: unconnected-(SW3-A-Pad1) -> SW_ML
- SW3 pad 2: unconnected-(SW3-B-Pad2) -> GND
- SW4 pad 1: unconnected-(SW4-A-Pad1) -> SW_MR
- SW4 pad 2: unconnected-(SW4-B-Pad2) -> GND
- SW5 pad 1: unconnected-(SW5-A-Pad1) -> SW_RT
- SW5 pad 2: unconnected-(SW5-B-Pad2) -> GND
- SW6 pad 1: unconnected-(SW6-A-Pad1) -> SW_RB
- SW6 pad 2: unconnected-(SW6-B-Pad2) -> GND
- SW7 pad 1: unconnected-(SW7-Pad1) -> XIAO_RST
- SW7 pad 2: unconnected-(SW7-Pad2) -> GND
- SW7 pad 3: unconnected-(SW7-Pad3) -> XIAO_RST
- SW7 pad 4: unconnected-(SW7-Pad4) -> GND
- SW8 pad 1: unconnected-(SW8-Pad1) -> Net-(J4-Pad1)
- SW8 pad 2: unconnected-(SW8-Pad2) -> VBAT_SW
- U2 pad 1: unconnected-(U2-+VCSEL-Pad1) -> Net-(U2-+VCSEL)
- U2 pad 10: unconnected-(U2-PASS_T-Pad10) -> Net-(U2-+VCSEL)
- U2 pad 11: unconnected-(U2-GND-Pad11) -> GND
- U2 pad 12: unconnected-(U2-CP-Pad12) -> Net-(U2-CP)
- U2 pad 13: unconnected-(U2-CN-Pad13) -> Net-(U2-CN)
- U2 pad 14: unconnected-(U2-VDD-Pad14) -> +1V8
- U2 pad 15: unconnected-(U2-XYLASER-Pad15) -> Net-(U2--VCSEL)
- U2 pad 16: unconnected-(U2--VCSEL-Pad16) -> Net-(U2--VCSEL)
- U2 pad 2: unconnected-(U2-SDIO-Pad2) -> PMW_SDIO
- U2 pad 3: unconnected-(U2-SCLK-Pad3) -> PMW_SCLK
- U2 pad 5: unconnected-(U2-NCS-Pad5) -> PMW_NCS
- U2 pad 6: unconnected-(U2-VDDIO-Pad6) -> +3V3
- U2 pad 7: unconnected-(U2-NRESET-Pad7) -> Net-(U2-NRESET)
- U2 pad 8: unconnected-(U2-MOTION-Pad8) -> PMW_MOTION
- U2 pad 9: unconnected-(U2-VCP-Pad9) -> Net-(U2-VCP)
- U3 pad 1: unconnected-(U3-VIN-Pad1) -> +3V3
- U3 pad 2: unconnected-(U3-GND-Pad2) -> GND
- U3 pad 3: unconnected-(U3-EN-Pad3) -> +3V3
- U3 pad 5: unconnected-(U3-VOUT-Pad5) -> +1V8

Commit message: update the pcb
Parts:
- C7: renamed from C2; value 1u -> 1u/X7R
- J1: renamed from J6; moved to B.Cu
- J2: renamed from J5; moved to B.Cu
- J3: renamed from J4; moved to B.Cu
- J6: renamed from J3; moved to B.Cu
- moved R1 71.5 mm to (173.0, 99.5)
- moved C3 68.4 mm to (168.8, 88.8)
- moved C4 68.4 mm to (168.8, 91.8)
- moved C5 65.4 mm to (164.2, 98.0), turned to -90 degrees
- moved C2 63.9 mm to (164.2, 102.2), turned to -90 degrees
- moved SW1 60.2 mm to (171.0, 61.9)
- moved C8 48.4 mm to (147.0, 106.0), turned to -90 degrees
- moved C7 47.4 mm to (145.0, 96.8), turned to -90 degrees
- moved C1 46.5 mm to (146.8, 91.7), turned to 90 degrees
- moved C6 41.7 mm to (137.5, 96.8), turned to -90 degrees
- moved U1 33.1 mm to (141.2, 96.8)
- moved SW8 27.7 mm to (140.8, 61.9)
- moved J3 17.0 mm to (117.2, 69.3), turned to 180 degrees
- turned J1 to 180 degrees
- turned J2 to 180 degrees
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- renumbered C7 to C1, C8 to C2, C4 to C3, C5 to C4, C3 to C5, C1 to C6, C6 to C8, J1 to J4, J2 to J5, SW8 to SW1, SW3 to SW2, SW4 to SW3, SW2 to SW4, SW1 to SW6, SW6 to SW7, SW7 to SW8, U3 to U1, U1 to U3
Connections:
- net Net-(J4-Pad1) renamed +BATT
- net VBAT_SW renamed +BAT_SW
- J5 pad 3: +3.3V -> +3V3

Commit message: update the pcb
Parts:
- moved J3 28.8 mm to (118.5, 98.0)
- moved R1 25.7 mm to (148.0, 93.6), turned to 90 degrees
- moved C6 20.2 mm to (152.2, 110.5)
- moved C7 20.2 mm to (159.8, 110.5)
- moved U1 20.2 mm to (156.0, 110.5)
- moved C1 6.91 mm to (148.0, 98.5), turned to -90 degrees
- moved C4 4.86 mm to (164.0, 92.5), turned to -90 degrees
- moved C3 4.40 mm to (166.5, 92.5), turned to -90 degrees
- moved C8 2.69 mm to (148.0, 103.5), turned to 90 degrees
- moved C5 0.56 mm to (164.0, 97.5)
- moved C2 0.32 mm to (164.0, 102.5)

Commit message: update the pcb
Parts:
- moved J6 41.6 mm to (160.5, 82.5), turned to -90 degrees
- moved J1 35.9 mm to (154.0, 82.5), turned to -90 degrees
- moved J2 32.4 mm to (151.0, 82.5), turned to -90 degrees
- moved J3 20.8 mm to (139.0, 94.5)
Other:
- board text added: "360mAh 20.5 x 38 x 5.8 mm"
- board text added: "620mAh 20.5 x 42 x 8.8 mm"
- board text added: "620mAh 22.5 x 50 x 6.3 mm"
Changed lines of the file:
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@@
 	(footprint "Adept_BLE_footprints:Pad_3x2mm"
 		(layer "B.Cu")
-		(at 119 87.648 180)
+		(at 151 82.5 -90)
 		(descr "Pad 3x2mm")
 		(tags "pad SMD")
 		(property "Reference" "J2"
-			(at 0 2.5 0)
+			(at 0 2.5 90)
 			(unlocked yes)
 			(layer "B.SilkS")
@@
 		)
 		(property "Value" "Conn_01x01_Pad"
-			(at -16 11 0)
+			(at -16 11 90)
 			(unlocked yes)
 			(layer "B.Fab")
@@
 		)
 		(property "Datasheet" ""
-			(at 0 0 0)
+			(at 0 0 90)
 			(unlocked yes)
 			(layer "B.Fab")
@@
 		)
 		(property "Description" "Generic connector, single row, 01x01"
-			(at 0 0 0)
+			(at 0 0 90)
 			(unlocked yes)
 			(layer "B.Fab")
@@
 		)
 		(property "MFR-PN" ""
-			(at 0 0 0)
+			(at 0 0 90)
 			(unlocked yes)
 			(layer "B.Fab")
@@
 		)
 		(property "DST-PN" ""
-			(at 0 0 0)
+			(at 0 0 90)
 			(unlocked yes)
 			(layer "B.Fab")
@@
 		(attr through_hole)
 		(fp_text user "${REFERENCE}"
-			(at 0 -2.5 0)
+			(at 0 -2.5 90)
 			(unlocked yes)
 			(layer "B.Fab")
@@
 		)
 		(pad "1" smd roundrect
-			(at 0 0 180)
+			(at 0 0 270)
 			(size 3 2)
 			(layers "B.Cu" "B.Mask" "B.Paste")
@@
 	(footprint "Adept_BLE_footprints:Pad_3x2mm"
 		(layer "B.Cu")
-		(at 119 90.648 180)
+		(at 154 82.5 -90)
 		(descr "Pad 3x2mm")
 		(tags "pad SMD")
 		(property "Reference" "J1"
-			(at 0 2.5 0)
+			(at 0 2.5 90)
 			(unlocked yes)
 			(layer "B.SilkS")
@@
 		)
 		(property "Value" "Conn_01x01_Pad"
-			(at -16 11 0)
+			(at -16 11 90)
 			(unlocked yes)
 			(layer "B.Fab")
@@
 		)
 		(property "Datasheet" ""
-			(at 0 0 0)
+			(at 0 0 90)
 			(unlocked yes)
 			(layer "B.Fab")
@@
 		)
 		(property "Description" "Generic connector, single row, 01x01"
-			(at 0 0 0)
+			(at 0 0 90)
 			(unlocked yes)
 			(layer "B.Fab")
@@
 		)
 		(property "MFR-PN" ""
-			(at 0 0 0)
+			(at 0 0 90)
 			(unlocked yes)
 			(layer "B.Fab")
@@
 		)
 		(property "DST-PN" ""
-			(at 0 0 0)
+			(at 0 0 90)
 			(unlocked yes)
 			(layer "B.Fab")
@@
 		(attr through_hole)
 		(fp_text user "${REFERENCE}"
-			(at 0 -2.5 0)
+			(at 0 -2.5 90)
 			(unlocked yes)
 			(layer "B.Fab")
@@
 		)
 		(pad "1" smd roundrect
-			(at 0 0 180)
+			(at 0 0 270)
 			(size 3 2)
 			(layers "B.Cu" "B.Mask" "B.Paste")
@@
 	(footprint "Adept_BLE_footprints:Pad_3x2mm"
 		(layer "B.Cu")
-		(at 119 84.648 180)
+		(at 160.5 82.5 -90)
 		(descr "Pad 3x2mm")
 		(tags "pad SMD")
 		(property "Reference" "J6"
-			(at 0 2.5 0)
+			(at 0 2.5 90)
 			(unlocked yes)
 			(layer "B.SilkS")
@@
 		)
 		(property "Value" "Conn_01x01_Pad"
-			(at -16 11 0)
+			(at -16 11 90)
 			(unlocked yes)
 			(layer "B.Fab")
@@
 		)
 		(property "Datasheet" ""
-			(at 0 0 0)
+			(at 0 0 90)
 			(unlocked yes)
 			(layer "B.Fab")
@@
 		)
 		(property "Description" "Generic connector, single row, 01x01"
-			(at 0 0 0)
+			(at 0 0 90)
 			(unlocked yes)
 			(layer "B.Fab")
@@
 		)
 		(property "MFR-PN" ""
-			(at 0 0 0)
+			(at 0 0 90)
 			(unlocked yes)
 			(layer "B.Fab")
@@
 		)
 		(property "DST-PN" ""
-			(at 0 0 0)
+			(at 0 0 90)
 			(unlocked yes)
 			(layer "B.Fab")
@@
 		(attr through_hole)
 		(fp_text user "${REFERENCE}"
-			(at 0 -2.5 0)
+			(at 0 -2.5 90)
 			(unlocked yes)
 			(layer "B.Fab")
@@
 		)
 		(pad "1" smd roundrect
-			(at 0 0 180)
+			(at 0 0 270)
 			(size 3 2)
 			(layers "B.Cu" "B.Mask" "B.Paste")
@@
 	(footprint "Adept_BLE_footprints:S2B-PH-K"
 		(layer "B.Cu")
-		(at 118.5 98.05 180)
+		(at 139 94.55 180)
 		(descr "side-entry, 2mm pitch, JST PH series connector")
 		(tags "connector JST PH horizontal")
@@
 		)
 	)
+	(gr_rect
+		(start 76.25 151.5)
+		(end 96.75 189.5)
+		(stroke
+			(width 0.1)
+			(type default)
+		)
+		(fill no)
+		(layer "Dwgs.User")
+	)
+	(gr_rect
+		(start 51.25 147.5)
+		(end 71.75 189.5)
+		(stroke
+			(width 0.1)
+			(type default)
+		)
+		(fill no)
+		(layer "Dwgs.User")
+	)
+	(gr_rect
+		(start 24.25 139.5)
+		(end 46.75 189.5)
+		(stroke
+			(width 0.1)
+			(type default)
+		)
+		(fill no)
+		(layer "Dwgs.User")
+	)
 	(gr_line
 		(start 127.8 125)
@@
 		(layer "Edge.Cuts")
 	)
+	(gr_text "620mAh\n20.5 x 42 x 8.8 mm"
+		(at 51.25 189.5 0)
+		(layer "Dwgs.User")
+		(effects
+			(font
+				(size 1 1)
+				(thickness 0.15)
+			)
+			(justify left bottom)
+		)
+	)
+	(gr_text "360mAh\n20.5 x 38 x 5.8 mm"
+		(at 76.25 189.5 0)
+		(layer "Dwgs.User")
+		(effects
+			(font
+				(size 1 1)
+				(thickness 0.15)
+			)
+			(justify left bottom)
+		)
+	)
+	(gr_text "620mAh\n22.5 x 50 x 6.3 mm"
+		(at 24.25 189.5 0)
+		(layer "Dwgs.User")
+		(effects
+			(font
+				(size 1 1)
+				(thickness 0.15)
+			)
+			(justify left bottom)
+		)
+	)
+	(group ""
+		(members "aa3df980-3ba6-4245-82c8-fc36678bd883" "e48cc0a2-c5b5-4365-95af-007ca08aa3ef")
+	)
+	(group ""
+		(members "c3082bf9-9b91-4615-bda5-0f2f8f6fcd18" "f12a983a-8df9-4b38-a061-6cac962805ff")
+	)
+	(group ""
+		(members "65bba196-21bc-4818-bc8e-2aea8fbea6a7" "ea12f3ae-f3be-4bac-96f9-d5b7e7a5f1f1")
+	)
 	(embedded_fonts no)
