File: Hardware/Adept_BLE.kicad_pcb (KiCad board)
At the start: 2 copper layers, 62 x 65.2 mm, 26 parts, among them J1 Conn_01x01_Pad, J2 Conn_01x01_Pad, J3 Conn_01x02_Pin, J4 Conn_01x07_Pad, J5 Conn_01x07_Pad, J6 Conn_01x01_Pad, SW1 PCM12SMTR, SW2 D2LS-21, SW3 D2LS-21, SW4 D2LS-21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

Commit message: update the pcb
Parts:
- moved J3 2.06 mm to (138.5, 96.5)
- moved C1 1.50 mm to (148.0, 97.0)
- moved C8 1.00 mm to (148.0, 104.5), turned to -90 degrees
- moved SW1 0.75 mm to (171.0, 61.1)
- moved SW8 0.75 mm to (140.8, 61.1)
- moved J1 0.50 mm to (154.0, 83.0)
- moved J2 0.50 mm to (151.0, 83.0)
- moved J6 0.50 mm to (160.5, 83.0)
- moved R1 0.50 mm to (148.0, 93.1), turned to -90 degrees
Connections:
- net +BAT_SW renamed +BATT_SW
- J4 pad 1: unconnected-(J4-Pin_1-Pad1) -> SW_LB
- J4 pad 2: SW_LB -> SW_LT
- J4 pad 3: SW_LT -> SW_ML
- J4 pad 4: SW_ML -> PMW_SDIO
- J4 pad 5: SW_MR -> PMW_SCLK
- J4 pad 6: SW_RT -> PMW_NCS
- J4 pad 7: SW_RB -> PMW_MOTION
- J5 pad 4: PMW_MOTION -> unconnected-(J5-Pin_4-Pad4)
- J5 pad 5: PMW_SDIO -> SW_MR
- J5 pad 6: PMW_SCLK -> SW_RT
- J5 pad 7: PMW_NCS -> SW_RB
- SW1 pad 1: +BATT -> unconnected-(SW1-Pad1)
- SW1 pad 3: unconnected-(SW1-Pad3) -> +BATT
Routing:
- net +3V3: track 0.00 -> 112.3 mm, vias 0 -> 4
- net SW_LB: track 0.00 -> 79.5 mm
- net SW_RB: track 0.00 -> 79.3 mm
- net +BATT: track 0.00 -> 64.9 mm
- net Net-(U2-+VCSEL): track 0.00 -> 54.8 mm
- net XIAO_RST: track 0.00 -> 52.5 mm
- net +BATT_SW: track 0.00 -> 42.2 mm
- net PMW_SDIO: track 0.00 -> 40.0 mm
- net PMW_SCLK: track 0.00 -> 35.8 mm
- net PMW_NCS: track 0.00 -> 33.1 mm
- net SW_RT: track 0.00 -> 20.7 mm
- net +1V8: track 0.00 -> 19.7 mm
- net SW_LT: track 0.00 -> 19.1 mm
- net PMW_MOTION: track 0.00 -> 18.7 mm
- net SW_MR: track 0.00 -> 7.85 mm
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Other:
- board size 62 x 65.2 mm -> 62 x 66 mm
