File: Hardware/nrf52840.kicad_sch (KiCad schematic)
At the start: 11 parts, among them J1 Conn_01x07_Pad, J2 Conn_01x07_Pad, J3 Conn_01x01_Pad, SW1 D2LS-21, SW2 D2LS-21, SW3 D2LS-21, SW4 D2LS-21, SW5 D2LS-21, SW6 D2LS-21, SW7 EVQPUC02K, U1 XIAO-nRF52840-SMD

Commit message: update the schematics
Parts:
- added J4: Conn_01x02_Pin, Adept_BLE_footprints:S2B-PH-K, symbol Adept_BLE_symbols:Conn_01x02_Pin
- added J5, J6: Conn_01x01_Pad, Adept_BLE_footprints:Pad_3x2mm, symbol Adept_BLE_symbols:Conn_01x01_Pad
- added SW8: PCM12SMTR, Adept_BLE_footprints:PCM12SMTR, symbol Adept_BLE_symbols:PCM12SMTR
- J3: footprint (none) -> Adept_BLE_footprints:Pad_3x2mm
Connections:
- net SW_RT: now reaches SW5.1 (A)
- net SW_RT: now also J1.6 (Pin_6), U1.6 (P0.05_A5_D5_SCL)
- net GND: now reaches SW5.2 (B)
- net GND: now also J2.2 (Pin_2), SW1.2 (B), SW2.2 (B), SW3.2 (B), SW4.2 (B), SW6.2 (B), SW7.2, SW7.4, U1.13 (GND), U1.21 (GND), J4.2, J6.1
- net XIAO_RST: now reaches SW7.1
- net XIAO_RST: now also J3.1, SW7.3, U1.17 (RESET)
- net SW_LB: now reaches J1.2 (Pin_2)
- net SW_LB: now also SW1.1 (A), U1.2 (P0.03_A1_D1)
- net SW_LT: now reaches J1.3 (Pin_3)
- net SW_LT: now also SW2.1 (A), U1.3 (P0.28_A2_D2)
- net SW_ML: now reaches J1.4 (Pin_4)
- net SW_ML: now also SW3.1 (A), U1.4 (P0.29_A3_D3)
- net SW_MR: now reaches J1.5 (Pin_5)
- net SW_MR: now also SW4.1 (A), U1.5 (P0.04_A4_D4_SDA)
- net SW_RB: now reaches J1.7 (Pin_7)
- net SW_RB: now also SW6.1 (A), U1.7 (P1.11_D6_TX)
- net PMW_SDIO: now reaches U1.10 (P1.14_D9_MISO)
- net PMW_SDIO: now also J2.5 (Pin_5)
- net PMW_MOTION: now reaches U1.11 (P1.15_D10_MOSI)
- net PMW_MOTION: now also J2.4 (Pin_4)
- net +3.3V: now reaches U1.12 (3V3)
- net +3.3V: now also J2.3 (Pin_3)
- net VBAT_SW: now reaches U1.22 (BAT)
- net VBAT_SW: now also J5.1, SW8.2
- net PMW_NCS: now reaches U1.8 (P1.12_D7_RX)
- net PMW_NCS: now also J2.7 (Pin_7)
- net PMW_SCLK: now reaches U1.9 (P1.13_D8_SCK)
- net PMW_SCLK: now also J2.6 (Pin_6)
- new net: J4.1, SW8.1
- no-connect marks 0 -> 10
Other:
- moved on the sheet: J1, J2, J3, SW1, SW2, SW3, SW4, SW5, SW6, SW7, U1

Commit message: update the schematics
Parts:
- renumbered J6 to J1, J5 to J2, J4 to J3, J1 to J4, J2 to J5, J3 to J6, SW8 to SW1, SW3 to SW2, SW4 to SW3, SW2 to SW4, SW1 to SW6, SW6 to SW7, SW7 to SW8, U1 to U3
Connections:
- net +BATT: now reaches J3.1, SW1.1
- net +3.3V renamed +3V3
- net VBAT_SW renamed +BAT_SW
Other:
- moved on the sheet: J1, J3

Commit message: add power flags to the schematics
Other:
- moved on the sheet: J1

Commit message: nrf52840.kicad_sch: update name of global label
Connections:
- net +BAT_SW renamed +BATT_SW
Changed lines of the file:
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@@
 		)
 	)
-	(global_label "+BAT_SW"
+	(global_label "+BATT_SW"
 		(shape input)
 		(at 223.52 116.84 0)
@@
 		)
 		(property "Intersheetrefs" "${INTERSHEET_REFS}"
-			(at 235.0323 116.84 0)
+			(at 235.9999 116.84 0)
 			(effects
 				(font
@@
 		)
 	)
-	(global_label "+BAT_SW"
+	(global_label "+BATT_SW"
 		(shape input)
 		(at 109.22 49.53 0)
@@
 		)
 		(property "Intersheetrefs" "${INTERSHEET_REFS}"
-			(at 120.7323 49.53 0)
-			(effects
-				(font
+			(at 121.6999 49.53 0)
+			(effects
+				(font

Commit message: update the schematics
Connections:
- net +BATT: now also SW1.3; no longer SW1.1
- net PMW_MOTION: now also J4.7 (Pin_7); no longer J5.4 (Pin_4)
- net PMW_NCS: now also J4.6 (Pin_6); no longer J5.7 (Pin_7)
- net PMW_SCLK: now also J4.5 (Pin_5); no longer J5.6 (Pin_6)
- net PMW_SDIO: now also J4.4 (Pin_4); no longer J5.5 (Pin_5)
- net SW_LB: now also J4.1 (Pin_1); no longer J4.2 (Pin_2)
- net SW_LT: now also J4.2 (Pin_2); no longer J4.3 (Pin_3)
- net SW_ML: now also J4.3 (Pin_3); no longer J4.4 (Pin_4)
- net SW_MR: now also J5.5 (Pin_5); no longer J4.5 (Pin_5)
- net SW_RB: now also J5.7 (Pin_7); no longer J4.7 (Pin_7)
- net SW_RT: now also J5.6 (Pin_6); no longer J4.6 (Pin_6)
